Commit message: Update robot assets and configuration for RoverX_Suspension_Test
- Updated chassis part and STL file with new microversion and ID.
- Added new parts: head_camera, knuckle_lf, knuckle_lm, knuckle_lr, knuckle_rf, knuckle_rm, knuckle_rr, rocker_arm_l, rocker_arm_r, wheel_lf, wheel_lm, wheel_lr, wheel_rf, wheel_rm, wheel_rr with corresponding STL files.
- Modified rocker_arm_left and rocker_arm_right parts to new microversion.
- Updated robot configuration in config.json with new URL and joint definitions.
- Enhanced robot.urdf with new visual and collision elements for added parts.
- Removed outdated robot.xml and scene.xml files.
- Updated Python virtual environment configuration.
- Added pybullet to requirements for enhanced simulation capabilities.

File: my-robot/robot.urdf (robot description, URDF)
Before this commit: robot C:\Users\r.canovas\REPOS\RoveX-Lab\my-robot, 1 links, 0 joints
Links:
- removed link chassis
- added link assembly_rover_v1, mass 1187.5; collision mesh filename=package://assets\bogie_arm_l.stl; collision mesh filename=package://assets\bogie_arm_r.stl

Commit message: Update robot asset

File: my-robot/robot.urdf (robot description, URDF)
Before this commit: robot RoverX_Suspension_Test, 1 links, 0 joints
Links:
- removed link assembly_rover_v1
- added link chassis, mass 1187.5; collision mesh filename=package://assets\bogie_arm_l.stl; collision mesh filename=package://assets\bogie_arm_r.stl
